Commit message: update piper_l piper_h urdf

File: piper_h_description/urdf/piper_h_description_d435.urdf (robot description, URDF)
Before this commit: robot piper_l_camera, 13 links, 12 joints
Links:
- link camera_link: geometry collision box size=0.02505 0.09 0.025; visual mesh filename=package://realsense2_description/meshes/d435.dae

File: piper_h_description/urdf/piper_h_description_d435_dark.urdf (robot description, URDF)
Before this commit: robot piper_l_camera, 13 links, 12 joints
Links:
- link Link1: mass 0.104656591084326 -> 0.095130320813071; geometry collision mesh filename=package://piper_h_description/meshes/dark_dae/link1.dae; visual mesh filename=package://piper_h_description/meshes/dark_dae/link1.dae
- link Link2: mass 0.289829779851577 -> 0.297349969020434; geometry collision mesh filename=package://piper_h_description/meshes/dark_dae/link2.dae; visual mesh filename=package://piper_h_description/meshes/dark_dae/link2.dae
- link Link3: mass 0.144963320053385 -> 0.139005088174055; geometry collision mesh filename=package://piper_h_description/meshes/dark_dae/link3.dae; visual mesh filename=package://piper_h_description/meshes/dark_dae/link3.dae
- link Link4: mass 0.063036548689954 -> 0.0625155037542606; geometry collision mesh filename=package://piper_h_description/meshes/dark_dae/link4.dae; visual mesh filename=package://piper_h_description/meshes/dark_dae/link4.dae
- link Link5: mass 0.069099989781007 -> 0.0683301439531726; geometry collision mesh filename=package://piper_h_description/meshes/dark_dae/link5.dae; visual mesh filename=package://piper_h_description/meshes/dark_dae/link5.dae
- link Link6: mass 0.00563228459599247 -> 0.851169543242842; geometry collision mesh filename=package://piper_h_description/meshes/dae/gripper_base_100_v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; visual mesh filename=package://piper_h_description/meshes/dae/gripper_base_100_v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
- link Link7: mass 0.0 -> None; geometry collision mesh filename=package://piper_h_description/meshes/dae/link7.dae; visual mesh filename=package://piper_h_description/meshes/dae/link7.dae
- link Link8: geometry collision mesh filename=package://piper_h_description/meshes/dae/link8.dae; visual mesh filename=package://piper_h_description/meshes/dae/link8.dae
- link base_link: mass 0.228506683240186 -> 0.17076936349368; geometry collision mesh filename=package://piper_h_description/meshes/dark_dae/base_link.dae; visual mesh filename=package://piper_h_description/meshes/dark_dae/base_link.dae
- link camera_stand_link: geometry collision mesh filename=package://piper_h_description/meshes/dae/realsense_mid_stan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; visual mesh filename=package://piper_h_description/meshes/dae/realsense_mid_stan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
Joints:
- joint joint2: origin xyz=0 0 0 rpy=1.5708 -0.10598 3.1416 -> xyz=0 0 0 rpy=1.5708 -0.13674 3.1416
- joint joint3: origin xyz=0.33823 0 0 rpy=0 0 -1.8325 -> xyz=0.28508 0 0 rpy=0 0 -1.8796
- joint joint4: axis 0 0 1 -> -0.087161 0 0.99619; origin xyz=0 -0.3215 0 rpy=1.5708 0 0.1557 -> xyz=0 -0.25666 0 rpy=1.5708 0 0.17203
- joint joint6: axis 0 0 1 -> -0.087161 0 0.99619; origin xyz=0 -0.091 0 rpy=1.5708 0 0 -> xyz=0 -0.096 0 rpy=1.5708 0 0.0

File: piper_l_description/urdf/piper_l_description_d435_dark.urdf (robot description, URDF)
Before this commit: robot piper_l_camera, 13 links, 12 joints
Links:
- link Link1: geometry collision mesh filename=package://piper_l_description/meshes/dark_dae/link1.dae; visual mesh filename=package://piper_l_description/meshes/dark_dae/link1.dae
- link Link2: geometry collision mesh filename=package://piper_l_description/meshes/dark_dae/link2.dae; visual mesh filename=package://piper_l_description/meshes/dark_dae/link2.dae
- link Link3: geometry collision mesh filename=package://piper_l_description/meshes/dark_dae/link3.dae; visual mesh filename=package://piper_l_description/meshes/dark_dae/link3.dae
- link Link4: geometry collision mesh filename=package://piper_l_description/meshes/dark_dae/link4.dae; visual mesh filename=package://piper_l_description/meshes/dark_dae/link4.dae
- link Link5: geometry collision mesh filename=package://piper_l_description/meshes/dark_dae/link5.dae; visual mesh filename=package://piper_l_description/meshes/dark_dae/link5.dae
- link base_link: geometry collision mesh filename=package://piper_l_description/meshes/dark_dae/base_link.dae; visual mesh filename=package://piper_l_description/meshes/dark_dae/base_link.dae
