Commit message: fixed urdf

File: piper_h_description/urdf/piper_h_description.xacro (robot description, xacro)
@@ -446,5 +446,5 @@
         </visual>
         <collision>
-            <origin xyz="0.0 0.0 0.0" rpy="0.0 0.0 0.0"/>
+            <origin xyz="0.0 0.0 0.0" rpy="0.0 3.14 1.57"/>
             <geometry>
                 <mesh filename="package://piper_h_description/meshes/dae/realsense_mid_stand_v2.dae" />

File: piper_l_description/urdf/piper_l_description.xacro (robot description, xacro)
@@ -446,5 +446,5 @@
         </visual>
         <collision>
-            <origin xyz="0.0 0.0 0.0" rpy="0.0 0.0 0.0"/>
+            <origin xyz="0.0 0.0 0.0" rpy="0.0 3.14 1.57"/>
             <geometry>
                 <mesh filename="package://piper_l_description/meshes/dae/realsense_mid_stand_v2.dae" />

File: piper_x_description/urdf/piper_x_description_d435.urdf (robot description, URDF)
Before this commit: robot piper_x_camera, 13 links, 12 joints
Links:
- link Link7: mass 0.0 -> 0.0264822021416248

Commit message: fixed urdf inertia

File: piper_h_description/urdf/piper_h_description.xacro (robot description, xacro)
@@ -8,16 +8,13 @@
     name="base_link">
     <inertial>
-      <origin
-        xyz="-0.0116216679858881 4.15788440943184E-05 0.0410845423187343"
-        rpy="0 0 0" />
-      <mass
-        value="0.17076936349368" />
-      <inertia
-        ixx="0.000228123208400866"
-        ixy="1.38955464051488E-07"
-        ixz="6.65141446336986E-06"
-        iyy="0.00027812842789125"
-        iyz="1.65175257145242E-07"
-        izz="0.000229266732859796" />
+      <origin xyz="-0.00347 -0.00012 0.04283" rpy="0 0 0"/>
+      <mass value="1.07"/>
+      <inertia
+          ixx="0.00099887"
+          ixy="0.00000194"
+          ixz="0.00000613"
+          iyy="0.00112771"
+          iyz="0.00000201"
+          izz="0.00096552" />
     </inertial>
     <visual>
@@ -48,16 +45,13 @@
     name="Link1">
     <inertial>
-      <origin
-        xyz="0.000898972809391425 -0.0017128345134696 -0.00895795324198079"
-        rpy="0 0 0" />
-      <mass
-        value="0.095130320813071" />
-      <inertia
-        ixx="3.89303819225542E-05"
-        ixy="2.71827364740144E-07"
-        ixz="1.78296584027163E-07"
-        iyy="5.60153481205046E-05"
-        iyz="1.02032883575856E-07"
-        izz="4.65461363833488E-05" />
+      <origin xyz="0.00038 -0.00039 -0.00317" rpy="0 0 0"/>
+      <mass value="0.71"/>
+      <inertia
+          ixx="0.00049803"
+          ixy="0.00000022"
+          ixz="0.00000810"
+          iyy="0.00040527"
+          iyz="0.00000116"
+          izz="0.00045753" />
     </inertial>
     <visual>
@@ -102,16 +96,13 @@
     name="Link2">
     <inertial>
-      <origin
-        xyz="0.175058051795962 -0.013263959401964 0.00160398731659567"
-        rpy="0 0 0" />
-      <mass
-        value="0.297349969020434" />
-      <inertia
-        ixx="0.000164919085428283"
-        ixy="6.39135842640096E-05"
-        ixz="-1.43495991521534E-06"
-        iyy="0.00163150429985587"
-        iyz="-1.15776231590507E-06"
-        izz="0.00168482164179664" />
+      <origin xyz="0.21849 -0.00875 0.00126" rpy="0 0 0"/>
+      <mass value="1.16"/>
+      <inertia
+          ixx="0.00103112"
+          ixy="0.00035994"
+          ixz="0.00012698"
+          iyy="0.01204356"
+          iyz="0.00000492"
+          izz="0.01188565" />
     </inertial>
     <visual>
@@ -156,16 +147,13 @@
     name="Link3">
     <inertial>
-      <origin
-        xyz="-0.00937198976084005 -0.116255702062803 -0.000655711046030733"
-        rpy="0 0 0" />
-      <mass
-        value="0.139005088174055" />
-      <inertia
-        ixx="0.000138596904431255"
-        ixy="-3.43992762936895E-07"
-        ixz="3.78558835970272E-07"
-        iyy="4.71404976476514E-05"
-        iyz="9.97047138050079E-07"
-        izz="0.000149219114996657" />
+      <origin xyz="-0.00778 -0.14512 -0.00047" rpy="0 0 0"/>
+      <mass value="0.55"/>
+      <inertia
+          ixx="0.00285399"
+          ixy="0.00008683"
+          ixz="0.00000260"
+          iyy="0.00025517"
+          iyz="0.00004073"
+          izz="0.00280819" />
     </inertial>
     <visual>
@@ -210,16 +198,13 @@
     name="Link4">
     <inertial>
-      <origin
-        xyz="0.00120008498546645 0.00402105386550108 -0.00901261181081513"
-        rpy="0 0 0" />
-      <mass
-        value="0.0625155037542606" />
-      <inertia
-        ixx="4.34001804299788E-05"
-        ixy="-1.78247237961623E-07"
-        ixz="7.9877981542642E-07"
-        iyy="3.77270563878061E-05"
-        iyz="3.92168392419924E-07"
-        izz="3.65881057070137E-05" />
+      <origin xyz="0.00051 -0.00091 -0.00395" rpy="0 0 0"/>
+      <mass value="0.36"/>
+      <inertia
+        ixx="0.00018477"
+        ixy="0.00000115"
+        ixz="0.00000323"
+        iyy="0.00016906"
+        iyz="0.00000674"
+        izz="0.00015871" />
     </inertial>
     <visual>
@@ -258,5 +243,5 @@
       link="Link4" />
     <axis
-      xyz="-0.087161 0 0.99619" />
+      xyz="0 0 1" />
     <limit lower="-1.832" upper="1.832" effort="100" velocity="3" />
   </joint>
@@ -264,16 +249,13 @@
     name="Link5">
     <inertial>
-      <origin
-        xyz="-9.76421424187524E-05 -0.0495078447416577 -0.0069183293653338"
-        rpy="0 0 0" />
-      <mass
-        value="0.0683301439531726" />
-      <inertia
-        ixx="8.08932317895225E-05"
-        ixy="2.20176838731191E-07"
-        ixz="5.56694167592644E-08"
-        iyy="4.13226227161016E-05"
-        iyz="1.71025553076376E-05"
-        izz="7.62573282419664E-05" />
+      <origin xyz="0.00015 -0.06349 -0.00253" rpy="0 0 0"/>
+      <mass value="0.38"/>
+      <inertia
+        ixx="0.00030399"
+        ixy="0.00000167"
+        ixz="0.00000011"
+        iyy="0.00016834"
+        iyz="0.00004817"
+        izz="0.00029057" />
     </inertial>
     <visual>
@@ -318,16 +300,13 @@
     name="Link6">
     <inertial>
-      <origin
-        xyz="0.0769862132705599 0.0288041655584747 -0.162335527696906"
-        rpy="0 0 0" />
-      <mass
-        value="0.851169543242842" />
-      <inertia
-        ixx="0.00204979841659076"
-        ixy="-3.46794622727557E-05"
-        ixz="-0.000104197916276416"
-        iyy="0.00210041391526329"
-        iyz="-0.000112551398932383"
-        izz="0.000469888685422321" />
+      <origin xyz="0 0 -0.00351" rpy="0 0 0"/>
+      <mass value="0.01"/>
+      <inertia
+        ixx="0.00000064"
+        ixy="0"
+        ixz="0"
+        iyy="0.00000064"
+        iyz="0"
+        izz="0.00000106"/>
     </inertial>
     <visual>
@@ -359,5 +338,5 @@
     type="revolute">
     <origin
-      xyz="0 -0.096 0"
+      xyz="0 -0.1 0"
       rpy="1.5708 0 0.0" />
     <parent
@@ -366,5 +345,5 @@
       link="Link6" />
     <axis
-      xyz="-0.087161 0 0.99619" />
+      xyz="0 0 1" />
     <limit lower="-3.14" upper="3.14" effort="100" velocity="3" />
   </joint>
@@ -372,5 +351,5 @@
   <visual>
     <inertial>
-      <origin rpy="0 0 0" xyz="0.000277816920932317 0.0467673824063769 -0.00921030054508036"/>
+      <origin rpy="0 0 0" xyz="0.000277816920932317 -0.0467673824063769 -0.00921030054508036"/>
       <mass value="0.0264822021416248"/>
       <inertia ixx="9.99779119357223E-06" ixy="-1.57542283433504E-07" ixz="2.71367446701359E-08" iyy="6.17952441557932E-06" iyz="1.58939319453383E-06" izz="1.4210192754512E-05"/>

File: piper_h_description/urdf/piper_h_description_d435.urdf (robot description, URDF)
Before this commit: robot piper_l_camera, 13 links, 12 joints
Links:
- link Link1: mass 0.095130320813071 -> 0.71
- link Link2: mass 0.297349969020434 -> 1.16
- link Link3: mass 0.139005088174055 -> 0.55
- link Link4: mass 0.0625155037542606 -> 0.36
- link Link5: mass 0.0683301439531726 -> 0.38
- link Link6: mass 0.851169543242842 -> 0.01
- link base_link: mass 0.17076936349368 -> 1.07
- link camera_link: geometry collision box size=0.02505 0.09 0.025; visual mesh filename=file:///home/agilex/piper_ws/install/realsense2_description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
Joints:
- joint joint4: axis -0.087161 0 0.99619 -> 0 0 1
- joint joint6: axis -0.087161 0 0.99619 -> 0 0 1; origin xyz=0 -0.096 0 rpy=1.5708 0 0.0 -> xyz=0 -0.1 0 rpy=1.5708 0 0.0

File: piper_h_description/urdf/piper_h_description_d435_dark.urdf (robot description, URDF)
Before this commit: robot piper_l_camera, 13 links, 12 joints
Links:
- link Link1: mass 0.095130320813071 -> 0.71; geometry collision mesh filename=package://piper_h_description/meshes/dae/dark_dae/link1.dae; visual mesh filename=package://piper_h_description/meshes/dae/dark_dae/link1.dae
- link Link2: mass 0.297349969020434 -> 1.16; geometry collision mesh filename=package://piper_h_description/meshes/dae/dark_dae/link2.dae; visual mesh filename=package://piper_h_description/meshes/dae/dark_dae/link2.dae
- link Link3: mass 0.139005088174055 -> 0.55; geometry collision mesh filename=package://piper_h_description/meshes/dae/dark_dae/link3.dae; visual mesh filename=package://piper_h_description/meshes/dae/dark_dae/link3.dae
- link Link4: mass 0.0625155037542606 -> 0.36; geometry collision mesh filename=package://piper_h_description/meshes/dae/dark_dae/link4.dae; visual mesh filename=package://piper_h_description/meshes/dae/dark_dae/link4.dae
- link Link5: mass 0.0683301439531726 -> 0.38; geometry collision mesh filename=package://piper_h_description/meshes/dae/dark_dae/link5.dae; visual mesh filename=package://piper_h_description/meshes/dae/dark_dae/link5.dae
- link Link6: mass 0.851169543242842 -> 0.01
- link base_link: mass 0.17076936349368 -> 1.07; geometry collision mesh filename=package://piper_h_description/meshes/dae/dark_dae/base_link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; visual mesh filename=package://piper_h_description/meshes/dae/dark_dae/base_link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
Joints:
- joint joint4: axis -0.087161 0 0.99619 -> 0 0 1
- joint joint6: axis -0.087161 0 0.99619 -> 0 0 1; origin xyz=0 -0.096 0 rpy=1.5708 0 0.0 -> xyz=0 -0.1 0 rpy=1.5708 0 0.0

File: piper_l_description/urdf/piper_l_description.xacro (robot description, xacro)
@@ -8,16 +8,13 @@
     name="base_link">
     <inertial>
-      <origin
-        xyz="-0.00868903062596066 -7.81380379250471E-05 0.0446229676471226"
-        rpy="0 0 0" />
-      <mass
-        value="0.228506683240186" />
-      <inertia
-        ixx="0.000187231110737863"
-        ixy="-1.08010529187549E-07"
-        ixz="7.71183528612253E-06"
-        iyy="0.000204010911651774"
-        iyz="1.70367399031094E-07"
-        izz="0.00023064619033588" />
+      <origin xyz="-0.00347 -0.00012 0.04283" rpy="0 0 0"/>
+      <mass value="1.07"/>
+      <inertia
+          ixx="0.00099887"
+          ixy="0.00000194"
+          ixz="0.00000613"
+          iyy="0.00112771"
+          iyz="0.00000201"
+          izz="0.00096552" />
     </inertial>
     <visual>
@@ -48,16 +45,13 @@
     name="Link1">
     <inertial>
-      <origin
-        xyz="0.000817078696798893 0.00114472671573105 -0.00814265146610774"
-        rpy="0 0 0" />
-      <mass
-        value="0.104656591084326" />
-      <inertia
-        ixx="3.99694684501781E-05"
-        ixy="2.71846206160129E-07"
-        ixz="1.78275886199695E-07"
-        iyy="5.78589658643876E-05"
-        iyz="1.01977672018063E-07"
-        izz="4.75851844139222E-05" />
+      <origin xyz="0.00201 -0.00220 -0.02127" rpy="0 0 0"/>
+      <mass value="0.11"/>
+      <inertia
+          ixx="0.00011279"
+          ixy="0.00000011"
+          ixz="0.00000186"
+          iyy="0.00007274"
+          iyz="0.00000781"
+          izz="0.00011091" />
     </inertial>
     <visual>
@@ -102,21 +96,18 @@
     name="Link2">
     <inertial>
-      <origin
-        xyz="0.214411452554835 -0.0136807991474291 0.00265923105206891"
-        rpy="0 0 0" />
-      <mass
-        value="0.289829779851577" />
-      <inertia
-        ixx="0.000159609737372076"
-        ixy="8.49438511625834E-05"
-        ixz="-8.73341391348404E-07"
-        iyy="0.00182424524515505"
-        iyz="-1.7222217649261E-06"
-        izz="0.00188778950006189" />
-    </inertial>
-    <visual>
-      <origin
-        xyz="0 0 0"
-        rpy="0 0 0" />
+      <origin xyz="0.25986 -0.00913 0.00237" rpy="0 0 0"/>
+      <mass value="1.16"/>
+      <inertia
+          ixx="0.00096865"
+          ixy="0.00041154"
+          ixz="0.00005836"
+          iyy="0.01629404"
+          iyz="0.00001694"
+          izz="0.01628996" />
+    </inertial>
+    <visual>
+      <origin
+        xyz="0 0 0"
+        rpy="0 0.0 0" />
       <geometry>
         <mesh
@@ -144,5 +135,5 @@
     <origin
       xyz="0 0 0"
-      rpy="1.5708 -0.10598 3.1416" />
+      rpy="1.5708 0.0 3.1416" />
     <parent
       link="Link1" />
@@ -156,16 +147,13 @@
     name="Link3">
     <inertial>
-      <origin
-        xyz="-0.00911397384332024 -0.149791842909887 -0.000591510024110218"
-        rpy="0 0 0" />
-      <mass
-        value="0.144963320053385" />
-      <inertia
-        ixx="0.000284000764414434"
-        ixy="6.61776597268393E-06"
-        ixz="3.88642213881568E-07"
-        iyy="4.88134965842348E-05"
-        iyz="8.80027301936097E-07"
-        izz="0.000297733639002112" />
+      <origin xyz="-0.00726 -0.19029 -0.00045" rpy="0 0 0"/>
+      <mass value="0.59"/>
+      <inertia
+          ixx="0.00558278"
+          ixy="0.00018354"
+          ixz="0.00000254"
+          iyy="0.00026568"
+          iyz="0.00005267"
+          izz="0.00554212" />
     </inertial>
     <visual>
@@ -210,16 +198,13 @@
     name="Link4">
     <inertial>
-      <origin
-        xyz="0.0010653905699945 0.00476990191039629 -0.00995810184233214"
-        rpy="0 0 0" />
-      <mass
-        value="0.063036548689954" />
-      <inertia
-        ixx="1.68358640686144E-05"
-        ixy="-1.51073528999065E-08"
-        ixz="-3.61196055919328E-07"
-        iyy="2.79335598814104E-05"
-        iyz="1.18113194001076E-07"
-        izz="1.85339684805634E-05" />
+      <origin xyz="0.00054 -0.00162 -0.00399" rpy="0 0 0"/>
+      <mass value="0.37"/>
+      <inertia
+          ixx="0.00017066"
+          ixy="0.00000129"
+          ixz="0.00000316"
+          iyy="0.00017128"
+          iyz="0.00000775"
+          izz="0.00014437" />
     </inertial>
     <visual>
@@ -252,5 +237,5 @@
     <origin
       xyz="0 -0.3215 0"
-      rpy="1.5708 0 0.1557" />
+      rpy="1.5708 0 0.0" />
     <parent
       link="Link3" />
@@ -264,16 +249,13 @@
     name="Link5">
     <inertial>
-      <origin
-        xyz="-5.62618579153795E-05 -0.0453229588602131 -0.00689048082401968"
-        rpy="0 0 0" />
-      <mass
-        value="0.069099989781007" />
-      <inertia
-        ixx="1.94244470320096E-05"
-        ixy="-3.01270043465718E-08"
-        ixz="-1.82908713601451E-08"
-        iyy="2.97665185121334E-05"
-        iyz="1.74803886281955E-07"
-        izz="2.43073597160068E-05" />
+      <origin xyz="0.0002 -0.06142 -0.00257" rpy="0 0 0"/>
+      <mass value="0.38"/>
+      <inertia
+          ixx="0.00029534"
+          ixy="0.00000167"
+          ixz="0.00000016"
+          iyy="0.00016988"
+          iyz="0.00005020"
+          izz="0.00028334" />
     </inertial>
     <visual>
@@ -306,5 +288,5 @@
     <origin
       xyz="0 0 0"
-      rpy="-1.5708 -0.087272 0" />
+      rpy="-1.5708 0.0 0" />
     <parent
       link="Link4" />
@@ -370,4 +352,17 @@
   </joint>
 <link name="Link7">
+  <inertial>
+  <origin
+      xyz="0.000277816920932317 -0.0467673824063769 -0.00921030054508036"
+      rpy="0 0 0" />
+  <mass value="0.0264822021416248" />
+  <inertia
+      ixx="9.99779119357223E-06"
+      ixy="-1.57542283433504E-07"
+      ixz="2.71367446701359E-08"
+      iyy="6.17952441557932E-06"
+      iyz="1.58939319453383E-06"
+      izz="1.4210192754512E-05" />
+  </inertial>
   <visual>
     <geometry>
@@ -383,9 +378,4 @@
     </geometry>
   </collision>
-  <inertial>
-    <mass value="0.0"/>
-    <origin xyz="0.0 0.0 0.0" rpy="0.0 0.0 0.0"/>
-    <inertia ixx="0.0" ixy="0.0" ixz="0.0" iyy="0.0" iyz="0.0" izz="0.0"/>
-  </inertial>
 </link>
     <joint name="joint7" type="prismatic">

File: piper_l_description/urdf/piper_l_description_d435.urdf (robot description, URDF)
Before this commit: robot piper_l_camera, 13 links, 12 joints
Links:
- link Link1: mass 0.104656591084326 -> 0.11
- link Link2: mass 0.289829779851577 -> 1.16
- link Link3: mass 0.144963320053385 -> 0.59
- link Link4: mass 0.063036548689954 -> 0.37
- link Link5: mass 0.069099989781007 -> 0.38
- link Link7: mass 0.0 -> 0.0264822021416248
- link base_link: mass 0.228506683240186 -> 1.07
Joints:
- joint joint2: origin xyz=0 0 0 rpy=1.5708 -0.10598 3.1416 -> xyz=0 0 0 rpy=1.5708 0.0 3.1416
- joint joint4: origin xyz=0 -0.3215 0 rpy=1.5708 0 0.1557 -> xyz=0 -0.3215 0 rpy=1.5708 0 0.0
- joint joint5: origin xyz=0 0 0 rpy=-1.5708 -0.087272 0 -> xyz=0 0 0 rpy=-1.5708 0.0 0

File: piper_l_description/urdf/piper_l_description_d435_dark.urdf (robot description, URDF)
Before this commit: robot piper_l_camera, 13 links, 12 joints
Links:
- link Link1: mass 0.104656591084326 -> 0.11; geometry collision mesh filename=package://piper_l_description/meshes/dae/dark_dae/link1.dae; visual mesh filename=package://piper_l_description/meshes/dae/dark_dae/link1.dae
- link Link2: mass 0.289829779851577 -> 1.16; geometry collision mesh filename=package://piper_l_description/meshes/dae/dark_dae/link2.dae; visual mesh filename=package://piper_l_description/meshes/dae/dark_dae/link2.dae
- link Link3: mass 0.144963320053385 -> 0.59; geometry collision mesh filename=package://piper_l_description/meshes/dae/dark_dae/link3.dae; visual mesh filename=package://piper_l_description/meshes/dae/dark_dae/link3.dae
- link Link4: mass 0.063036548689954 -> 0.37; geometry collision mesh filename=package://piper_l_description/meshes/dae/dark_dae/link4.dae; visual mesh filename=package://piper_l_description/meshes/dae/dark_dae/link4.dae
- link Link5: mass 0.069099989781007 -> 0.38; geometry collision mesh filename=package://piper_l_description/meshes/dae/dark_dae/link5.dae; visual mesh filename=package://piper_l_description/meshes/dae/dark_dae/link5.dae
- link Link7: mass 0.0 -> 0.0264822021416248
- link base_link: mass 0.228506683240186 -> 1.07; geometry collision mesh filename=package://piper_l_description/meshes/dae/dark_dae/base_link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; visual mesh filename=package://piper_l_description/meshes/dae/dark_dae/base_link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
Joints:
- joint joint2: origin xyz=0 0 0 rpy=1.5708 -0.10598 3.1416 -> xyz=0 0 0 rpy=1.5708 0.0 3.1416
- joint joint4: origin xyz=0 -0.3215 0 rpy=1.5708 0 0.1557 -> xyz=0 -0.3215 0 rpy=1.5708 0 0.0
- joint joint5: origin xyz=0 0 0 rpy=-1.5708 -0.087272 0 -> xyz=0 0 0 rpy=-1.5708 0.0 0
