Commit message: fixed urdf inertia

File: piper_x_description/urdf/piper_x_description.xacro (robot description, xacro)
@@ -5,59 +5,50 @@
 <robot xmlns:xacro="http://www.ros.org/wiki/xacro" name="piper_x_camera">
 <xacro:include filename="$(find realsense2_description)/urdf/test_d435_camera.urdf.xacro" />
-  <link
+<link
     name="base_link">
-    <inertial>
-      <origin
-        xyz="-0.0085443 4.8839E-05 0.044762"
-        rpy="0 0 0" />
-      <mass
-        value="0.47421" />
+  <inertial>
+    <origin xyz="-0.00347 -0.00012 0.04283" rpy="0 0 0"/>
+    <mass value="1.07"/>
+    <inertia
+        ixx="0.00099887"
+        ixy="0.00000194"
+        ixz="0.00000613"
+        iyy="0.00112771"
+        iyz="0.00000201"
+        izz="0.00096552" />
+  </inertial>
+    <visual>
+      <origin
+        xyz="0 0 0"
+        rpy="0 0 0" />
+      <geometry>
+        <mesh
+          filename="package://piper_x_description/meshes/dae/base_Link.dae" />
+      </geometry>
+      <material
+        name="">
+        <color
+          rgba="0.59216 0.61961 0.65098 1" />
+      </material>
+    </visual>
+    <collision>
+      <origin
+        xyz="0 0 0"
+        rpy="0 0 0" />
+      <geometry>
+        <mesh
+          filename="package://piper_x_description/meshes/dae/base_Link.dae" />
+      </geometry>
+    </collision>
+  </link>
+  <link
+    name="Link1">
+    <inertial>
+      <origin xyz="0.00065 0.00006 -0.00325" rpy="0 0 0" />
+      <mass value="0.71" />
       <inertia
-        ixx="0.00044509"
-        ixy="5.5896E-07"
-        ixz="1.9736E-05"
-        iyy="0.00049109"
-        iyz="7.1578E-07"
-        izz="0.00055319" />
-    </inertial>
-    <visual>
-      <origin
-        xyz="0 0 0"
-        rpy="0 0 0" />
-      <geometry>
-        <mesh
-          filename="package://piper_x_description/meshes/dae/base_Link.dae" />
-      </geometry>
-      <material
-        name="">
-        <color
-          rgba="0.59216 0.61961 0.65098 1" />
-      </material>
-    </visual>
-    <collision>
-      <origin
-        xyz="0 0 0"
-        rpy="0 0 0" />
-      <geometry>
-        <mesh
-          filename="package://piper_x_description/meshes/dae/base_Link.dae" />
-      </geometry>
-    </collision>
-  </link>
-  <link
-    name="Link1">
-    <inertial>
-      <origin
-        xyz="0.0011378 -0.0021698 -0.014112"
-        rpy="0 0 0" />
-      <mass
-        value="0.16975" />
-      <inertia
-        ixx="6.466E-05"
-        ixy="7.2374E-07"
-        ixz="5.1556E-08"
-        iyy="8.8951E-05"
-        iyz="1.0827E-07"
-        izz="8.3142E-05" />
+        ixx="0.00050503" ixy="0.00000291" ixz="0.00000889"
+        iyy="0.00040309" iyz="0.00000225"
+        izz="0.00045932" />
     </inertial>
     <visual>
@@ -106,16 +97,13 @@
     name="Link2">
     <inertial>
-      <origin
-        xyz="0.21036 -0.01651 0.0015283"
-        rpy="0 0 0" />
-      <mass
-        value="0.37783" />
-      <inertia
-        ixx="0.00022199"
-        ixy="3.2631E-05"
-        ixz="-6.2643E-06"
-        iyy="0.0019854"
-        iyz="-3.0109E-06"
-        izz="0.0020664" />
+      <origin xyz="0.21854 -0.00853 0.00234" rpy="0 0 0"/>
+      <mass value="1.16"/>
+    <inertia
+        ixx="0.0010067"
+        ixy="0.0003653"
+        ixz="0.00004563"
+        iyy="0.01202556"
+        iyz="0.00001515"
+        izz="0.01193901" />
     </inertial>
     <visual>
@@ -159,16 +147,13 @@
     name="Link3">
     <inertial>
-      <origin
-        xyz="0.15119 -0.0060622 0.0013657"
-        rpy="0 0 0" />
-      <mass
-        value="0.28003" />
-      <inertia
-        ixx="9.0698E-05"
-        ixy="8.6875E-07"
-        ixz="-2.0769E-06"
-        iyy="0.00035668"
-        iyz="1.1019E-06"
-        izz="0.00039114" />
+      <origin xyz="0.20190 -0.00415 -0.00114" rpy="0 0 0"/>
+      <mass value="0.67"/>
+    <inertia
+        ixx="0.00032229"
+        ixy="0.00029258"
+        ixz="0.00001566"
+        iyy="0.00628179"
+        iyz="0.00000371"
+        izz="0.00623643" />
     </inertial>
     <visual>
@@ -217,16 +202,13 @@
     name="Link4">
     <inertial>
-      <origin
-        xyz="0.041795 -0.032887 -0.0088781"
-        rpy="0 0 0" />
-      <mass
-        value="0.1211" />
-      <inertia
-        ixx="5.6173E-05"
-        ixy="-8.0853E-07"
-        ixz="-5.604E-07"
-        iyy="6.2662E-05"
-        iyz="-1.3477E-07"
-        izz="6.8648E-05" />
+      <origin xyz="0.06593 -0.04751 -0.00274" rpy="0 0 0"/>
+      <mass value="0.4"/>
+    <inertia
+        ixx="0.00030498"
+        ixy="0.00014139"
+        ixz="0.00005955"
+        iyy="0.00036923"
+        iyz="0.00004930"
+        izz="0.00046330" />
     </inertial>
     <visual>
@@ -275,16 +257,13 @@
     name="Link5">
     <inertial>
-      <origin
-        xyz="0.0041507 0.00024807 -0.015852"
-        rpy="0 0 0" />
-      <mass
-        value="0.094498" />
-      <inertia
-        ixx="4.0846E-05"
-        ixy="5.2625E-08"
-        ixz="7.7998E-07"
-        iyy="2.5458E-05"
-        iyz="-2.0306E-07"
-        izz="3.3445E-05" />
+      <origin xyz="0.00005 -0.01299 -0.00417" rpy="0 0 0"/>
+      <mass value="0.35"/>
+    <inertia
+        ixx="0.00016058"
+        ixy="0.00000042"
+        ixz="0.00000003"
+        iyy="0.00017124"
+        iyz="0.00001836"
+        izz="0.00013440" />
     </inertial>
     <visual>
@@ -333,16 +312,13 @@
     name="Link6">
     <inertial>
-      <origin
-        xyz="4.4377E-07 -1.9614E-05 0.031556"
-        rpy="0 0 0" />
-      <mass
-        value="0.0061311" />
-      <inertia
-        ixx="5.1682E-07"
-        ixy="9.18E-25"
-        ixz="1.1291E-22"
-        iyy="5.1683E-07"
-        iyz="2.6088E-09"
-        izz="9.833E-07" />
+      <origin xyz="-0.00006 -0.00003 0.04448" rpy="0 0 0"/>
+      <mass value="0.52"/>
+    <inertia
+        ixx="0.00048224"
+        ixy="0.00000048"
+        ixz="0.00000136"
+        iyy="0.00059105"
+        iyz="0.00000208"
+        izz="0.00030728" />
     </inertial>
     <visual>
@@ -388,24 +364,32 @@
       velocity="10" />
   </joint>
-<link name="Link7">
-  <visual>
-    <geometry>
-      <mesh filename="package://piper_x_description/meshes/dae/J7.dae" />
-    </geometry>
-    <material name="LightGrey">
-      <color rgba="0.7 0.7 0.7 1.0"/>
-    </material>
-  </visual>
-  <collision>
-    <geometry>
-      <mesh filename="package://piper_x_description/meshes/dae/J7.dae" />
-    </geometry>
-  </collision>
-  <inertial>
-    <mass value="0.0"/>
-    <origin xyz="0.0 0.0 0.0" rpy="0.0 0.0 0.0"/>
-    <inertia ixx="0.0" ixy="0.0" ixz="0.0" iyy="0.0" iyz="0.0" izz="0.0"/>
-  </inertial>
-</link>
+  <link name="Link7">
+    <inertial>
+    <origin
+        xyz="0.000277816920932317 -0.0467673824063769 -0.00921030054508036"
+        rpy="0 0 0" />
+    <mass value="0.0264822021416248" />
+    <inertia
+        ixx="9.99779119357223E-06"
+        ixy="-1.57542283433504E-07"
+        ixz="2.71367446701359E-08"
+        iyy="6.17952441557932E-06"
+        iyz="1.58939319453383E-06"
+        izz="1.4210192754512E-05" />
+    </inertial>
+    <visual>
+      <geometry>
+        <mesh filename="package://piper_x_description/meshes/dae/J7.dae" />
+      </geometry>
+      <material name="LightGrey">
+        <color rgba="0.7 0.7 0.7 1.0"/>
+      </material>
+    </visual>
+    <collision>
+      <geometry>
+        <mesh filename="package://piper_x_description/meshes/dae/J7.dae" />
+      </geometry>
+    </collision>
+  </link>
     <joint name="joint7" type="prismatic">
         <origin xyz="0 0 0.13503" rpy="1.5708 0 1.5708" />

File: piper_x_description/urdf/piper_x_description_d435.urdf (robot description, URDF)
Before this commit: robot piper_x_camera, 13 links, 12 joints
Links:
- link Link1: mass 0.16975 -> 0.71
- link Link2: mass 0.37783 -> 1.16
- link Link3: mass 0.28003 -> 0.67
- link Link4: mass 0.1211 -> 0.4
- link Link5: mass 0.094498 -> 0.35
- link Link6: mass 0.0061311 -> 0.52
- link base_link: mass 0.47421 -> 1.07
