Commit message: 更正urdf

File: piper_h_description/urdf/piper_h_description copy.urdf (robot description, URDF)
Before this commit: robot piper_l_description, 7 links, 6 joints
Links:
- link Link1: mass 0.104656591084326 -> 0.71; geometry collision mesh filename=package://piper_h_description/meshes/Link1.STL; visual mesh filename=package://piper_h_description/meshes/Link1.STL
- link Link2: mass 0.289829779851577 -> 1.16; geometry collision mesh filename=package://piper_h_description/meshes/Link2.STL; visual mesh filename=package://piper_h_description/meshes/Link2.STL
- link Link3: mass 0.144963320053385 -> 0.55; geometry collision mesh filename=package://piper_h_description/meshes/Link3.STL; visual mesh filename=package://piper_h_description/meshes/Link3.STL
- link Link4: mass 0.063036548689954 -> 0.36; geometry collision mesh filename=package://piper_h_description/meshes/Link4.STL; visual mesh filename=package://piper_h_description/meshes/Link4.STL
- link Link5: mass 0.069099989781007 -> 0.38; geometry collision mesh filename=package://piper_h_description/meshes/Link5.STL; visual mesh filename=package://piper_h_description/meshes/Link5.STL
- link Link6: mass 0.00563228459599247 -> 0.01; geometry collision mesh filename=package://piper_h_description/meshes/Link6.STL; visual mesh filename=package://piper_h_description/meshes/Link6.STL
- link base_link: mass 0.228506683240186 -> 1.07; geometry collision mesh filename=package://piper_h_description/meshes/base_link.STL; visual mesh filename=package://piper_h_description/meshes/base_link.STL
Joints:
- joint joint1: limit lower=-2.618 upper=2.618 effort=100 velocity=3 -> lower=0 upper=0 effort=0 velocity=0
- joint joint2: limit lower=0 upper=3.14 effort=100 velocity=3 -> lower=0 upper=0 effort=0 velocity=0; origin xyz=0 0 0 rpy=1.5708 -0.1745 3.1416 -> xyz=0 0 0 rpy=1.5708 -0.13674 3.1416
- joint joint3: limit lower=-2.697 upper=0 effort=100 velocity=3 -> lower=0 upper=0 effort=0 velocity=0; origin xyz=0.33823 0 0 rpy=0 0 -1.8325 -> xyz=0.28508 0 0 rpy=0 0 -1.8796
- joint joint4: axis 0 0 1 -> -0.087161 0 0.99619; limit lower=-1.832 upper=1.832 effort=100 velocity=3 -> lower=0 upper=0 effort=0 velocity=0; origin xyz=0 -0.3215 0 rpy=1.5708 0 0.1557 -> xyz=0 -0.25666 0 rpy=1.5708 0 0.17203
- joint joint5: limit lower=-1.22 upper=1.22 effort=100 velocity=3 -> lower=0 upper=0 effort=0 velocity=0
- joint joint6: axis 0 0 1 -> -0.087161 0 0.99619; limit lower=-3.14 upper=3.14 effort=100 velocity=3 -> lower=0 upper=0 effort=0 velocity=0; origin xyz=0 -0.091 0 rpy=1.5708 0 0 -> xyz=0 -0.096 0 rpy=1.5708 0 0.087272

File: piper_l_description/urdf/piper_l_description copy.urdf (robot description, URDF)
Before this commit: robot piper_l_description, 7 links, 6 joints
Links:
- link Link1: mass 0.104656591084326 -> 0.11
- link Link2: mass 0.289829779851577 -> 1.16
- link Link3: mass 0.144963320053385 -> 0.59
- link Link4: mass 0.063036548689954 -> 0.37
- link Link5: mass 0.069099989781007 -> 0.38
- link base_link: mass 0.228506683240186 -> 1.07
Joints:
- joint joint2: origin xyz=0 0 0 rpy=1.5708 -0.1745 3.1416 -> xyz=0 0 0 rpy=1.5708 0.0 3.1416

File: piper_l_description/urdf/piper_l_description.xacro (robot description, xacro)
@@ -135,5 +135,5 @@
     <origin
       xyz="0 0 0"
-      rpy="1.5708 0.0 3.1416" />
+      rpy="1.5708 -0.1745 3.1416" />
     <parent
       link="Link1" />

File: piper_l_description/urdf/piper_l_description_d435.urdf (robot description, URDF)
Before this commit: robot piper_l_camera, 13 links, 12 joints
Joints:
- joint joint2: origin xyz=0 0 0 rpy=1.5708 0.0 3.1416 -> xyz=0 0 0 rpy=1.5708 -0.1745 3.1416

File: piper_l_description/urdf/piper_l_description_d435_dark.urdf (robot description, URDF)
Before this commit: robot piper_l_camera, 13 links, 12 joints
Joints:
- joint joint2: origin xyz=0 0 0 rpy=1.5708 0.0 3.1416 -> xyz=0 0 0 rpy=1.5708 -0.1745 3.1416

File: piper_x_description/urdf/piper_x_description_no_gripper.urdf (robot description, URDF)
Before this commit: robot piper_x_description, 9 links, 8 joints
Links:
- removed link Link6
- removed link Link7
- removed link Link8
- added link link6, mass 0.01; collision mesh filename=package://piper_x_description/meshes/link6.STL; visual mesh filename=package://piper_x_description/meshes/link6.STL
Joints:
- removed joint joint7
- removed joint joint8
