Commit message: update piper urdf

File: piper_description/urdf/piper_description_v100_realsense_camera_v2.urdf (robot description, URDF)
Before this commit: robot piper_camera, 13 links, 12 joints
Links:
- link camera_link: geometry collision box size=0.02505 0.09 0.025; visual mesh filename=file:///home/agilex/piper_ws/install/realsense2_description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

Commit message: update piper urdf

File: piper_description/urdf/piper_description_v100_realsense_camera_v2.urdf (robot description, URDF)
Before this commit: robot piper_camera, 13 links, 12 joints
Links:
- link camera_link: geometry collision box size=0.02505 0.09 0.025; visual mesh filename=package://realsense2_description/meshes/d435.dae
