Commit message: 修复 piper_description_v100_realsense_camera_v2_dark

File: piper_description/urdf/piper_description_v100_realsense_camera_v2_dark.urdf (robot description, URDF)
Before this commit: robot piper_camera, 13 links, 12 joints
Links:
- link link6: geometry collision mesh filename=package://piper_description/meshes/dae/link6_.dae; visual mesh filename=package://piper_description/meshes/dae/link6_.dae
- link link7: geometry collision mesh filename=package://piper_description/meshes/dae/link7.dae; visual mesh filename=package://piper_description/meshes/dae/link7.dae
- link link8: geometry collision mesh filename=package://piper_description/meshes/dae/link8.dae; visual mesh filename=package://piper_description/meshes/dae/link8.dae
