Commit message: add nero dae

File: nero_description/urdf/nero_description.urdf (robot description, URDF)
Before this commit: robot nero_description, 8 links, 7 joints
Links:
- link Link1: mass 0.24545463218233 -> 0.77
- link Link2: mass 0.340250343180855 -> 0.49
- link Link3: mass 0.359899395208716 -> 0.67
- link Link4: mass 0.164135315169796 -> 0.41
- link Link5: mass 0.26290365411796 -> 0.56
- link Link6: mass 0.0346374690978017 -> 0.31
