Commit message: 修改nero的惯量

File: nero_description/urdf/nero_description.xacro (robot description, xacro)
@@ -8,16 +8,7 @@
     name="base_link">
     <inertial>
-      <origin
-        xyz="-0.00963614954335565 0.00016786624100977 0.044860101664403"
-        rpy="0 0 0" />
-      <mass
-        value="0.487153985946125" />
-      <inertia
-        ixx="0.000448116331022417"
-        ixy="5.78111047127811E-07"
-        ixz="1.54743135248644E-05"
-        iyy="0.000492511294798627"
-        iyz="-4.11935494337721E-07"
-        izz="0.000552986424582884" />
+      <origin rpy="0 0 0" xyz="-0.00347 -0.00012 0.04283"/>
+      <mass value="1.07"/>
+      <inertia ixx="0.00099887" ixy="0.00000194" ixz="0.00000613" iyy="0.00112771" iyz="0.00000201" izz="0.00096552"/>
     </inertial>
     <visual>
@@ -97,7 +88,7 @@
     name="Link2">
     <inertial>
-      <origin xyz="-0.00011 -0.06072 0.00148" rpy="0 0 0" />
-      <mass value="0.49" />
-      <inertia ixx="0.00053808" ixy="0.00000079" ixz="0.00000009" iyy="0.00029435" iyz="0.00004088" izz="0.00040266" />
+      <origin xyz="0.0008 -0.0789 0.00112" rpy="0 0 0" />
+      <mass value="0.69" />
+      <inertia ixx="0.00201094" ixy="0.00002399" ixz="0.00000073" iyy="0.00063544" iyz="0.00005831" izz="0.00181944" />
     </inertial>
     <visual>
@@ -195,7 +186,7 @@
     name="Link4">
     <inertial>
-      <origin xyz="-0.00013 -0.05482 0.00132" rpy="0 0 0" />
-      <mass value="0.41" />
-      <inertia ixx="0.00031331" ixy="0.00000009" ixz="0.00000007" iyy="0.00013204" iyz="0.00001401" izz="0.00023930" />
+      <origin xyz="-0.00032 -0.05876 0.0007" rpy="0 0 0" />
+      <mass value="0.48" />
+      <inertia ixx="0.00054472" ixy="0.00000564" ixz="0.00000007" iyy="0.00026240" iyz="0.00001922" izz="0.00044249" />
     </inertial>
     <visual>
