Commit message: Update piper_x_description_no_gripper.urdf
Update piper_x_description_no_gripper.urdf

File: piper_x_description/urdf/piper_x_description_no_gripper.urdf (robot description, URDF)
Before this commit: robot piper_x_description, 7 links, 6 joints
Links:
- removed link link6
- added link Link6, mass 0.01; collision mesh filename=package://piper_x_description/meshes/link6.STL; visual mesh filename=package://piper_x_description/meshes/link6.STL
